File: schematic/stm32f407vgt/stm32f407vgt.kicad_pcb (KiCad board)
At the start: 2 copper layers, 31 parts

Commit message: ok
Parts:
- removed the 1_dot at (163.8, 119.4)
- removed the 1_dot at (164.3, 68.6)
- removed the 1_dot at (169.3, 68.6)
- removed the 1_dot at (84.1, 153.4)
- removed the 1_dot at (163.8, 116.8)
- removed the 1_dot at (108.3, 153.4)
- removed the 1_dot at (119.4, 153.4)
- removed the 1_dot at (86.4, 116.8)
- removed the 1_dot at (86.4, 119.4)
- removed the 1_dot at (163.8, 114.3)
- removed the 1_dot at (171.4, 74.7)
- removed the 1_dot at (162.6, 74.7)
- removed the 1_dot at (84.1, 157.5)
- added 1_dot: 1_dot, 1_dot, F.Cu at (44.5, 94.0)
- added 1_dot: 1_dot, 1_dot, F.Cu at (132.1, 132.1)
- added 1_dot: 1_dot, 1_dot, F.Cu at (127.0, 132.1)
- added 1_dot: 1_dot, 1_dot, F.Cu at (205.7, 94.0)
- added 1_dot: 1_dot, 1_dot, F.Cu at (205.7, 91.4)
- added 1_dot: 1_dot, 1_dot, F.Cu at (205.7, 88.9)
- added 1_dot: 1_dot, 1_dot, F.Cu at (82.5, 94.0)
- added 1_dot: 1_dot, 1_dot, F.Cu at (150.2, 128.0)
- added 1_dot: 1_dot, 1_dot, F.Cu at (161.3, 128.0)
- added 1_dot: 1_dot, 1_dot, F.Cu at (128.3, 91.4)
- added 1_dot: 1_dot, 1_dot, F.Cu at (128.3, 94.0)
- added 1_dot: 1_dot, 1_dot, F.Cu at (44.5, 132.1)
- added 1_dot: 1_dot, 1_dot, F.Cu at (82.5, 132.1)
- added 1_dot: 1_dot, 1_dot, F.Cu at (106.2, 105.3)
- added 1_dot: 1_dot, 1_dot, F.Cu at (106.2, 110.4)
- added 1_dot: 1_dot, 1_dot, F.Cu at (101.6, 131.8)
- added 1_dot: 1_dot, 1_dot, F.Cu at (106.7, 131.8)
- added 1_dot: 1_dot, 1_dot, F.Cu at (111.8, 131.8)
- added REF**: 16_pin, 16_pin, F.Cu at (66.0, 57.1)
- added REF**: 16_pin, 16_pin, F.Cu at (66.0, 52.1)
- moved 1_dot 49.0 mm to (181.6, 122.9)
- moved 1_dot 49.0 mm to (128.3, 96.5)
- moved REF** 49.0 mm to (125.7, 31.8)
- moved 1_dot 49.0 mm to (176.5, 122.9)
- moved REF** 49.0 mm to (171.4, 82.5)
- moved a9g 49.0 mm to (231.1, 78.7)
- moved jum5 49.0 mm to (130.8, 81.3)
- moved hum4 49.0 mm to (130.8, 108.0)
- moved jum8 49.0 mm to (221.0, 108.0)
- moved 1_dot 49.0 mm to (173.0, 128.0)
- moved 1_dot 49.0 mm to (184.2, 128.3)
- moved 1_dot 47.9 mm to (212.1, 25.2)
- moved 1_dot 47.9 mm to (217.2, 25.2)
- moved 1_dot 47.9 mm to (207.0, 25.2)
- moved 1_dot 41.9 mm to (252.0, 33.4)
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Routing:
- net (no net): track 2146.6 -> 2426.2 mm
Other:
- net class Default: trace_width 0.4 -> 1
- board text added: "Power for L298"
- board text added: "RES_200K"
- board text added: "photo_back"
- board text removed: "LED"
- board text removed: "RESISTOR"
- board text removed: "RES_100K"
- board text removed: "photo"

Commit message: ok
Parts:
- removed the 1_dot at (205.7, 94.0)
- removed the 1_dot at (205.7, 91.4)
- removed the 1_dot at (205.7, 88.9)
- removed the 1_dot at (150.2, 128.0)
- removed the 1_dot at (161.3, 128.0)
- removed the 1_dot at (128.3, 91.4)
- removed the 1_dot at (128.3, 94.0)
- added 1_dot: 1_dot, 1_dot, F.Cu at (204.5, 108.0)
- added 1_dot: 1_dot, 1_dot, F.Cu at (204.5, 105.4)
- added 1_dot: 1_dot, 1_dot, F.Cu at (204.5, 102.9)
- added 1_dot: 1_dot, 1_dot, F.Cu at (148.9, 142.0)
- added 1_dot: 1_dot, 1_dot, F.Cu at (160.0, 142.0)
- added 1_dot: 1_dot, 1_dot, F.Cu at (127.0, 105.4)
- added 1_dot: 1_dot, 1_dot, F.Cu at (127.0, 108.0)
- moved 1_dot 14.5 mm to (221.0, 39.1)
- moved 1_dot 14.5 mm to (215.9, 39.1)
- moved 1_dot 14.5 mm to (210.8, 39.1)
- moved 1_dot 14.0 mm to (104.9, 119.3)
- moved REF** 14.0 mm to (64.8, 71.1)
- moved REF** 14.0 mm to (64.8, 66.0)
- moved 1_dot 14.0 mm to (43.2, 108.0)
- moved 1_dot 14.0 mm to (130.8, 146.1)
- moved 1_dot 14.0 mm to (125.7, 146.1)
- moved 1_dot 14.0 mm to (250.8, 47.4)
- moved 1_dot 14.0 mm to (81.3, 108.0)
- moved 1_dot 14.0 mm to (175.3, 136.9)
- moved 1_dot 14.0 mm to (180.3, 136.9)
- moved 1_dot 14.0 mm to (182.9, 142.2)
- moved 1_dot 14.0 mm to (43.2, 146.1)
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Routing:
- net (no net): track 2426.2 -> 2424.4 mm
Other:
- board text added: "VDD_3.3v"
- board text added: "VDD_5v"
